File: splitter.sch (KiCad schematic (older format))
At the start: 3 parts, among them J1 NI68PinConnector, J2 NI68PinConnector, J3 PinHeaders

Commit message: added silk screen labels, post processed into gerber files
Connections:
- net labels added: FTLU6, P0.1
- net labels removed: P.1, TFLU6
Changed lines of the file:
@@
 FTLU5
 Text Label 1650 6650 0    60   ~ 12
-TFLU6
+FTLU6
 Text Label 1700 4050 0    60   ~ 12
 FTRU1
@@
 P0.6
 Text Label 2000 2350 0    60   ~ 0
-P.1
+P0.1
 Text Label 2000 2550 0    60   ~ 0
 P0.4
@@
 APFI_0
 Text Label 5800 3100 0    60   ~ 0
-P.1
+P0.1
 Text Label 5800 3000 0    60   ~ 0
 P0.3
@@
 UCrank
 Text Label 4600 3500 0    60   ~ 0
-TFLU6
+FTLU6
 Text Label 4600 3600 0    60   ~ 0
 FTRU4
